File: audio_dev_board/MCU.kicad_sch (KiCad schematic)
At the start: 36 parts, among them J1 TC2030, J2 USB_C_Receptacle_USB2.0_16P, SW1 SW_Push, U1 STM32H743VITx, U2 AMS1117-3.3, U3 USBLC6-2SC6, X1 32kHz768, X2 25Mhz

Commit message: bluhhh
Other:
- note added: "STM32"
- note added: "STM32 POWER + CRYSTALS"
- note added: "USB-C"
- moved on the sheet: C1, C10, C11, C12, C13, C14, C15, C16, C17, C18, C19, C2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
